File: 2024/Eagle/new_boards/main_board_0V5.sch (EAGLE design)
At the start: 5 parts

Commit message: .
Parts:
- added C1, C2: (no value), rcl:C-EUC0805
- added IR6: TSSP58038, TSOP4038:TSOP4038
- added OUT1_A, OUT2_A: (no value), wirepad:3,81/1,4
- added R5, R6, R7: (no value), rcl:R-EU_R0805
Connections:
- net N$8 renamed CS_A
- new net +5V: C1.1, R5.1, R6.1
- new net N$3: IR6.VS, R5.2
- new net N$6: C2.1, R7.1
- new net N$7: IR6.VO, R6.2, R7.2
- net GND: now also C1.2, C2.2, IR6.GND, R1.1, R2.1, R3.1, R4.1
- net N$11: now also OUT1_A.P
- net N$9: now also OUT2_A.P

Commit message: eagle
Parts:
- added C3, C4, C5, C6, C7, C8, C9: 100nF, rcl:C-EUC0805
- added D1, D2, D3, D4, D5, D6, D7, D8: OF-SMD2835Y, OF-SMD2835Y:OF-SMD2835Y
- added R10, R11, R12, R13, R14, R15, R8, R9: 330R, rcl:R-EU_R1206
- renumbered IR6 to IR1, MOTOR_D_DRV to U1, OUT1_A to PAD1, OUT2_A to PAD2
Connections:
- new net N$10: C3.1, C4.1, C5.1, C6.1, C7.1, C8.1, C9.1, D1.C, D2.C, D3.C, D4.C, D5.C, D6.C, D7.C, D8.C
- new net N$70: D2.A, R9.1
- new net N$71: D3.A, R10.1
- new net N$72: D4.A, R11.1
- new net N$73: D5.A, R12.1
- new net N$74: D6.A, R13.1
- new net N$75: D7.A, R14.1
- new net N$76: D8.A, R15.1
- new net N$8: D1.A, R8.1
- net +5V: now also C3.2, C4.2, C5.2, C6.2, C7.2, C8.2, C9.2, R10.2, R11.2, R12.2, R13.2, R14.2, R15.2, R8.2, R9.2
- net N$1: now also R4.2; no longer R1.2
- net N$2: now also R3.2; no longer R2.2
- net N$4: now also R1.2; no longer R4.2
- net N$5: now also R2.2; no longer R3.2

Commit message: eagle
Parts:
- added C10, C11, C12, C13, C14, C15, C16, C17, C48, C53: 100nF, rcl:C-EUC0805
- added C54: 470uF, rcl:CPOL-EU150CLZ-1010
- added D10, D11, D12, D13, D14, D15, D16, D9: OF-SMD2835Y, OF-SMD2835Y:OF-SMD2835Y
- added D35: SS34, SamacSys_Parts:SS34
- added IC1: CD74HC4067SM96, SamacSys_Parts:CD74HC4067SM96
- added IC3: AZ1117CH-3.3TRG1, AZ1117CH-3.3TRG1:AZ1117CH-3.3TRG1
- added L3: 33uH, SamacSys_Parts:7443551151
- added Q1, Q10, Q11, Q12, Q13, Q14, Q15, Q16, Q2, Q3, Q4, Q5, Q6, Q7, Q8, Q9: PT19-21B/L41/TR8, PT19-21B_L41_TR8:PT19-21B/L41/TR8
- added R16, R17, R18, R19, R20, R21, R22, R23: 330R, rcl:R-EU_R0805
- added R24, R25, R26, R27, R28, R29, R30, R31, R32, R33, R34, R35, R36, R37, R38, R39: 10k, rcl:R-EU_R0805
- added R40: 10K, rcl:R-TRIMM3314J
- added TP1, TP10, TP11, TP12, TP13, TP14, TP15, TP16, TP17, TP18, TP19, TP2, TP20, TP21, TP22, TP23, TP24, TP25, TP26, TP27, TP28, TP29, TP3, TP30, TP31, TP32, TP4, TP5, TP6, TP7, TP8, TP9: PTR1PAD1-13, testpad:PTR1PAD1-13
- added U2: MEGA_PRO_EMBED_CH340G_/_ATMEGA2560, MEGA_PRO_EMBED_CH340G___ATMEGA2560:MEGA_PRO_EMBED_CH340G_/_ATMEGA2560
- added U3, U4, U5: BH-18650-PC, BH-18650-PC:BH-18650-PC
- added U9: XL4005, XL4015:XL4015
- D3: SPICEPREFIX D -> (none)
- R10, R11, R12, R13, R14, R15, R8, R9: device rcl:R-EU_R1206 -> rcl:R-EU_R0805
Connections:
- new net +3V3: C15.1, C17.1, IC1.VCC, IC3.OUTPUT, IC3.VOUT
- new net LI0: Q1.C, Q10.C, Q11.C, Q12.C, Q13.C, Q14.C, Q15.C, Q16.C, Q2.C, Q3.C, Q4.C, Q5.C, Q6.C, Q7.C, Q8.C, Q9.C, R24.2, R25.2, R26.2, R27.2, R28.2, R29.2, R30.2, R31.2, R32.2, R33.2, R34.2, R35.2, R36.2, R37.2, R38.2, R39.2
- new net LIGHT_I0: IC1.I0, TP1.TP
- new net LIGHT_I1: IC1.I1, TP2.TP
- new net LIGHT_I10: IC1.I10, TP11.TP
- new net LIGHT_I11: IC1.I11, TP12.TP
- new net LIGHT_I12: IC1.I12, TP13.TP
- new net LIGHT_I13: IC1.I13, TP14.TP
- new net LIGHT_I14: IC1.I14, TP15.TP
- new net LIGHT_I15: IC1.I15, TP16.TP
- new net LIGHT_I16: TP17.TP
- new net LIGHT_I17: TP18.TP
- new net LIGHT_I18: TP19.TP
- new net LIGHT_I19: TP20.TP
- new net LIGHT_I2: IC1.I2, TP3.TP
- new net LIGHT_I20: TP21.TP
- new net LIGHT_I21: TP22.TP
- new net LIGHT_I22: TP23.TP
- new net LIGHT_I23: TP24.TP
- new net LIGHT_I24: TP25.TP
- new net LIGHT_I25: TP26.TP
- new net LIGHT_I26: TP27.TP
- new net LIGHT_I27: TP28.TP
- new net LIGHT_I28: TP29.TP
- new net LIGHT_I29: TP30.TP
- new net LIGHT_I3: IC1.I3, TP4.TP
- new net LIGHT_I30: TP31.TP
- new net LIGHT_I31: TP32.TP
- new net LIGHT_I4: IC1.I4, TP5.TP
- new net LIGHT_I5: IC1.I5, TP6.TP
- new net LIGHT_I6: IC1.I6, TP7.TP
- new net LIGHT_I7: IC1.I7, TP8.TP
- new net LIGHT_I8: IC1.I8, TP9.TP
- new net LIGHT_I9: IC1.I9, TP10.TP
- new net LIGHT_READ_A: IC1.COMMON_INPUT/OUTPUT
- new net LIGHT_SET_0: IC1.S0
- new net LIGHT_SET_1: IC1.S1
- new net LIGHT_SET_2: IC1.S2
- new net LIGHT_SET_3: IC1.S3
- new net N$13: D9.A, R16.1
- new net N$14: D10.A, R17.1
- new net N$16: D11.A, R18.1
- new net N$18: D12.A, R19.1
- new net N$20: D13.A, R20.1
- new net N$22: D14.A, R21.1
- new net N$24: D15.A, R22.1
- new net N$26: D16.A, R23.1
- new net N$28: D1.C, D10.C, D11.C, D12.C, D13.C, D14.C, D15.C, D16.C, D2.C, D3.C, D4.C, D5.C, D6.C, D7.C, D8.C, D9.C
- new net N$29: D35.K, L3.1, U9.SW
- new net N$30: C53.2, R40.S, U9.FB
- new net N$8: U4.-, U5.+
- net +12V: now also U9.EN, U9.VIN
- net +5V: now also C10.2, C11.2, C12.2, C13.2, C14.2, C16.1, C48.1, C53.1, C54.+, IC3.INPUT, L3.2, R16.2, R17.2, R18.2, R19.2, R20.2, R21.2, R22.2, R23.2, R24.1, R25.1, R26.1, R27.1, R28.1, R29.1, R30.1, R31.1, R32.1, R33.1, R34.1, R35.1, R36.1, R37.1, R38.1, R39.1, R40.A
- net GND: now also C10.1, C11.1, C12.1, C13.1, C14.1, C15.2, C16.2, C17.2, C3.1, C4.1, C48.2, C5.1, C54.-, C6.1, C7.1, C8.1, C9.1, D35.A, IC1.!E, IC1.GND, IC3.ADJ/GND, Q1.E, Q10.E, Q11.E, Q12.E, Q13.E, Q14.E, Q15.E, Q16.E, Q2.E, Q3.E, Q4.E, Q5.E, Q6.E, Q7.E, Q8.E, Q9.E, R40.E, U9.GND
- net N$10: now also U3.-, U4.+; no longer C3.1, C4.1, C5.1, C6.1, C7.1, C8.1, C9.1, D1.C, D2.C, D3.C, D4.C, D5.C, D6.C, D7.C, D8.C

Commit message: eagle
Parts:
- removed TP17, TP18, TP19, TP20, TP21, TP22, TP23, TP24, TP25, TP26, TP27, TP28, TP29, TP30, TP31, TP32: PTR1PAD1-13, testpad:PTR1PAD1-13
- added Q17: CSD19503KCS, CSD19503KCS:CSD19503KCS
- added Q52: BSS138, BSS138:BSS138
- added R41, R42: 10k, rcl:R-EU_R1206
Connections:
- net LIGHT_READ_A renamed LIGHT_READ
- net LIGHT_SET_0 renamed LS0
- net LIGHT_SET_1 renamed LS1
- net LIGHT_SET_2 renamed LS2
- net LIGHT_SET_3 renamed LS3
- removed net LIGHT_I0: IC1.I0, TP1.TP
- removed net LIGHT_I1: IC1.I1, TP2.TP
- removed net LIGHT_I10: IC1.I10, TP11.TP
- removed net LIGHT_I11: IC1.I11, TP12.TP
- removed net LIGHT_I12: IC1.I12, TP13.TP
- removed net LIGHT_I13: IC1.I13, TP14.TP
- removed net LIGHT_I14: IC1.I14, TP15.TP
- removed net LIGHT_I15: IC1.I15, TP16.TP
- removed net LIGHT_I16: TP17.TP
- removed net LIGHT_I17: TP18.TP
- removed net LIGHT_I18: TP19.TP
- removed net LIGHT_I19: TP20.TP
- removed net LIGHT_I2: IC1.I2, TP3.TP
- removed net LIGHT_I20: TP21.TP
- removed net LIGHT_I21: TP22.TP
- removed net LIGHT_I22: TP23.TP
- removed net LIGHT_I23: TP24.TP
- removed net LIGHT_I24: TP25.TP
- removed net LIGHT_I25: TP26.TP
- removed net LIGHT_I26: TP27.TP
- removed net LIGHT_I27: TP28.TP
- removed net LIGHT_I28: TP29.TP
- removed net LIGHT_I29: TP30.TP
- removed net LIGHT_I3: IC1.I3, TP4.TP
- removed net LIGHT_I30: TP31.TP
- removed net LIGHT_I31: TP32.TP
- removed net LIGHT_I4: IC1.I4, TP5.TP
- removed net LIGHT_I5: IC1.I5, TP6.TP
- removed net LIGHT_I6: IC1.I6, TP7.TP
- removed net LIGHT_I7: IC1.I7, TP8.TP
- removed net LIGHT_I8: IC1.I8, TP9.TP
- removed net LIGHT_I9: IC1.I9, TP10.TP
- new net +5V_UP: R41.2
- new net LED_EN: Q52.S, R42.1
- new net LI1: IC1.I1, Q2.C, R25.2, TP2.TP
- new net LI10: IC1.I10, Q11.C, R34.2, TP11.TP
- new net LI11: IC1.I11, Q12.C, R35.2, TP12.TP
- new net LI12: IC1.I12, Q13.C, R36.2, TP13.TP
- new net LI13: IC1.I13, Q14.C, R37.2, TP14.TP
- new net LI14: IC1.I14, Q15.C, R38.2, TP15.TP
- new net LI15: IC1.I15, Q16.C, R39.2, TP16.TP
- new net LI2: IC1.I2, Q3.C, R26.2, TP3.TP
- new net LI3: IC1.I3, Q4.C, R27.2, TP4.TP
- new net LI4: IC1.I4, Q5.C, R28.2, TP5.TP
- new net LI5: IC1.I5, Q6.C, R29.2, TP6.TP
- new net LI6: IC1.I6, Q7.C, R30.2, TP7.TP
- new net LI7: IC1.I7, Q8.C, R31.2, TP8.TP
- new net LI8: IC1.I8, Q9.C, R32.2, TP9.TP
- new net LI9: IC1.I9, Q10.C, R33.2, TP10.TP
- new net N$31: Q17.S, R10.2, R11.2, R12.2, R13.2, R14.2, R15.2, R16.2, R17.2, R18.2, R19.2, R20.2, R21.2, R22.2, R23.2, R8.2, R9.2
- new net N$32: Q17.G, Q52.D, R41.1
- net +12V: now also Q17.D
- net +3V3: no longer C17.1, IC1.VCC
- net +5V: now also C17.1, IC1.VCC, Q52.G, R42.2; no longer R10.2, R11.2, R12.2, R13.2, R14.2, R15.2, R16.2, R17.2, R18.2, R19.2, R20.2, R21.2, R22.2, R23.2, R8.2, R9.2
- net LI0: now also IC1.I0, TP1.TP; no longer Q10.C, Q11.C, Q12.C, Q13.C, Q14.C, Q15.C, Q16.C, Q2.C, Q3.C, Q4.C, Q5.C, Q6.C, Q7.C, Q8.C, Q9.C, R25.2, R26.2, R27.2, R28.2, R29.2, R30.2, R31.2, R32.2, R33.2, R34.2, R35.2, R36.2, R37.2, R38.2, R39.2
Other:
- moved on the sheet: C15, C16, C17, D1, D2, D3, D4, D5, D6, D7, D8, IC1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
