File: 2024/PCBs/tsopV2.brd (EAGLE design)
At the start: 69.9 x 69.9 mm, 36 parts, among them IC2 CD74HC4067SM96, Q1 BSS138

Commit message: tsop
Parts:
- added C14, C15, C16, C17: 100nF, rcl:C0805
- added IR13, IR14, IR15, IR16: TSSP58038, TSOP4038:TSOP
- moved IR12 126.2 mm to (29.4, -17.0), turned to 330 degrees
- moved IR11 107.9 mm to (17.0, -29.4), turned to 300 degrees
- moved IR3 102.8 mm to (17.0, 29.4), turned to 60 degrees
- moved IR2 102.1 mm to (29.4, 17.0), turned to 30 degrees
- moved IR4 97.1 mm to (0.00, 34.0), turned to 90 degrees
- moved IR1 94.4 mm to (34.0, 0.00)
- moved IR5 86.7 mm to (-17.0, 29.4), turned to 120 degrees
- moved IR10 85.1 mm to (0.00, -34.0), turned to 270 degrees
- moved IR6 76.1 mm to (-29.4, 17.0), turned to 150 degrees
- moved IR9 60.3 mm to (-17.0, -29.4), turned to 240 degrees
- moved IR8 37.5 mm to (-29.4, -17.0), turned to 210 degrees
- moved IR7 26.0 mm to (-34.0, 0.00), turned to 180 degrees
Connections:
- net +5V: now also C14.1, C15.1, C16.1, C17.1, IR13.VS, IR14.VS, IR15.VS, IR16.VS
- net GND: now also C14.2, C15.2, C16.2, C17.2, IR13.GND, IR14.GND, IR15.GND, IR16.GND
- net I10: now also IR14.VO, IR16.VO
- net I9: now also IR13.VO, IR15.VO
Other:
- board size 69.9 x 69.9 mm -> 73.7 x 73.7 mm
