File: 2024/PCBs/tsopV2.sch (EAGLE design)
At the start: 36 parts, among them IC2 CD74HC4067SM96, Q1 BSS138

Commit message: tsop
Parts:
- added C14, C15, C16, C17: 100nF, rcl:C-EUC0805
- added IR13, IR14, IR15, IR16: TSSP58038, TSOP4038:TSOP4038
Connections:
- net +5V: now also C14.1, C15.1, C16.1, C17.1, IR13.VS, IR14.VS, IR15.VS, IR16.VS
- net GND: now also C14.2, C15.2, C16.2, C17.2, IR13.GND, IR14.GND, IR15.GND, IR16.GND
- net I10: now also IR14.VO, IR16.VO
- net I9: now also IR13.VO, IR15.VO
