File: 2024/PCBs/top_PCB_V2.sch (EAGLE design)
At the start: 36 parts, among them IC2 CD74HC4067SM96, Q1 BSS138

Commit message: tsop
Parts:
- removed BLUE, GREEN, RED: (no value), jumper:SJ
- removed C10, C11, C12, C13, C7, C8, C9: 100nF, rcl:C-EUC0805
- removed CON: (no value), pinhead:PINHD-2X4
- removed IC2: CD74HC4067SM96, SamacSys_Parts:CD74HC4067SM96
- removed IR1, IR10, IR11, IR12, IR2, IR3, IR4, IR5, IR6, IR7, IR8, IR9: TSSP58038, TSOP4038:TSOP4038
- removed LED: LTST-G563ZEGBW, LTST-G563ZEGBW:LTST-G563ZEGBW
- removed Q1: BSS138, BSS138:BSS138
- removed R1: 330R, rcl:R-EU_R1206
- added ARDUINO_MEGA: MEGA_PRO_EMBED_CH340G_/_ATMEGA2560, MEGA_PRO_EMBED_CH340G___ATMEGA2560:MEGA_PRO_EMBED_CH340G_/_ATMEGA2560
- added BNO085: 4754, 4754:4754
- added DISPLAY: (no value), pinhead:PINHD-1X4
- added FUSE: (no value), rcl:R-EU_R1206
- added J2: XT60-M, XT60-M:XT60-M
- added MAIN_CONNECTOR: TST-120-02-S-D, TST-120-02-S-D:TST-120-02-S-D
- added MPU-6050: (no value), pinhead:PINHD-1X8
- added OS1, OS2: (no value), tcrt5000:TCRT5000
- added POWER_SWITCH: 100SP1T1B4M2QE, 100SP1T1B4M2QE:100SP1T1B4M2QE
- added R5: 330R, rcl:R-EU_R1206
- added R6, R7: 10K, rcl:R-EU_R1206
- added RESET, START: DTSM-6, switch-tact:DTSM-6
- added TSOP_0, TSOP_1: (no value), pinhead:PINHD-2X4
- added U$1: BNO055_ADAFRUIT, BNO055_Adafruit:BNO055_ADAFRUIT
- R2: value 330R -> 4k7
- R4: value 10K -> 4k7
Connections:
- removed net I0: IC2.I0, IR1.VO
- removed net I1: IC2.I1, IR2.VO
- removed net I10: IC2.I10, IR11.VO
- removed net I11: IC2.I11, IR12.VO
- removed net I12: IC2.I12
- removed net I13: IC2.I13
- removed net I14: IC2.I14
- removed net I15: IC2.I15
- removed net I2: IC2.I2, IR3.VO
- removed net I3: IC2.I3, IR4.VO
- removed net I4: IC2.I4, IR5.VO
- removed net I5: IC2.I5, IR6.VO
- removed net I6: IC2.I6, IR7.VO
- removed net I7: IC2.I7, IR8.VO
- removed net I8: IC2.I8, IR9.VO
- removed net I9: IC2.I9, IR10.VO
- removed net IR_READ: CON.2, IC2.COMMON_INPUT/OUTPUT
- removed net N$4: R3.2, RED.2
- removed net N$7: BLUE.1, GREEN.1, Q1.S, RED.1
- new net +12V: ARDUINO_MEGA.VIN, MAIN_CONNECTOR.10
- new net +3V3: MAIN_CONNECTOR.12, MAIN_CONNECTOR.14
- new net BALL_CHECK_0: ARDUINO_MEGA.A8, OS1.COLLECTOR, R2.1
- new net BALL_CHECK_1: ARDUINO_MEGA.A10, OS2.COLLECTOR, R4.1
- new net EN_A: ARDUINO_MEGA.D23, MAIN_CONNECTOR.03
- new net EN_B: ARDUINO_MEGA.D31, MAIN_CONNECTOR.11
- new net EN_C: ARDUINO_MEGA.D35, MAIN_CONNECTOR.19
- new net EN_D: ARDUINO_MEGA.D41, MAIN_CONNECTOR.27
- new net GYRO_SCL: ARDUINO_MEGA.D21, BNO085.SCL, DISPLAY.3, MPU-6050.3, U$1.P$5
- new net GYRO_SDA: ARDUINO_MEGA.D20, BNO085.SDA, DISPLAY.4, MPU-6050.4, U$1.P$4
- new net IN1_A: ARDUINO_MEGA.D25, MAIN_CONNECTOR.05
- new net IN1_B: ARDUINO_MEGA.D29, MAIN_CONNECTOR.13
- new net IN1_C: ARDUINO_MEGA.D37, MAIN_CONNECTOR.21
- new net IN1_D: ARDUINO_MEGA.D43, MAIN_CONNECTOR.29
- new net IN2_A: ARDUINO_MEGA.D27, MAIN_CONNECTOR.07
- new net IN2_B: ARDUINO_MEGA.D33, MAIN_CONNECTOR.15
- new net IN2_C: ARDUINO_MEGA.D39, MAIN_CONNECTOR.23
- new net IN2_D: ARDUINO_MEGA.D45, MAIN_CONNECTOR.31
- new net IR_READ_A: ARDUINO_MEGA.A12, TSOP_0.4
- new net IR_READ_B: ARDUINO_MEGA.A14, TSOP_1.4
- new net KICKER: ARDUINO_MEGA.D4, MAIN_CONNECTOR.01
- new net LED_ENABLE: ARDUINO_MEGA.D6, MAIN_CONNECTOR.08
- new net LIGHT_READ_A: ARDUINO_MEGA.A13, MAIN_CONNECTOR.04
- new net LIGHT_READ_B: ARDUINO_MEGA.A15, MAIN_CONNECTOR.06
- new net PWM_A: ARDUINO_MEGA.D3, MAIN_CONNECTOR.09
- new net PWM_B: ARDUINO_MEGA.D5, MAIN_CONNECTOR.17
- new net PWM_C: ARDUINO_MEGA.D7, MAIN_CONNECTOR.25
- new net PWM_D: ARDUINO_MEGA.D9, MAIN_CONNECTOR.33
- new net RESET_SWITCH: ARDUINO_MEGA.D2, R6.1, RESET.1, RESET.2
- new net START_SWITCH: ARDUINO_MEGA.D19, R7.1, START.1, START.2
- net +5V: now also BNO085.VIN, DISPLAY.2, MAIN_CONNECTOR.16, MAIN_CONNECTOR.18, MAIN_CONNECTOR.20, MAIN_CONNECTOR.22, MAIN_CONNECTOR.24, MAIN_CONNECTOR.26, MPU-6050.1, R2.2, R3.2, R4.2, R5.2, R6.2, R7.2, TSOP_0.1, TSOP_1.1, U$1.P$1; no longer C10.1, C11.1, C12.1, C13.1, C7.1, C8.1, C9.1, CON.1, IC2.VCC, IR1.VS, IR10.VS, IR11.VS, IR12.VS, IR2.VS, IR3.VS, IR4.VS, IR5.VS, IR6.VS, IR7.VS, IR8.VS, IR9.VS, Q1.D
- net GND: now also ARDUINO_MEGA.GND, BNO085.GND, DISPLAY.1, MAIN_CONNECTOR.28, MAIN_CONNECTOR.30, MAIN_CONNECTOR.32, MAIN_CONNECTOR.34, MAIN_CONNECTOR.36, MAIN_CONNECTOR.38, MAIN_CONNECTOR.40, MPU-6050.2, OS1.CATHODE, OS1.EMITTER, OS2.CATHODE, OS2.EMITTER, RESET.3, RESET.4, START.3, START.4, TSOP_0.8, TSOP_1.8; no longer C10.2, C11.2, C12.2, C13.2, C7.2, C8.2, C9.2, CON.6, IC2.!E, IC2.GND, IR1.GND, IR10.GND, IR11.GND, IR12.GND, IR2.GND, IR3.GND, IR4.GND, IR5.GND, IR6.GND, IR7.GND, IR8.GND, IR9.GND, LED.1, LED.2, LED.3, R4.1
- net LED_UP: now also TSOP_0.6, TSOP_1.6; no longer CON.4, Q1.G, R4.2
- net LIGHT_SET_0: now also ARDUINO_MEGA.D28, MAIN_CONNECTOR.35, TSOP_0.3, TSOP_1.3; no longer CON.3, IC2.S0
- net LIGHT_SET_1: now also ARDUINO_MEGA.D26, MAIN_CONNECTOR.37, TSOP_0.5, TSOP_1.5; no longer CON.5, IC2.S1
- net LIGHT_SET_2: now also ARDUINO_MEGA.D24, MAIN_CONNECTOR.39, TSOP_0.7, TSOP_1.7; no longer CON.7, IC2.S2
- net LIGHT_SET_3: now also ARDUINO_MEGA.D22, MAIN_CONNECTOR.02, TSOP_0.2, TSOP_1.2; no longer CON.8, IC2.S3
- net N$1: now also FUSE.2, POWER_SWITCH.2; no longer LED.6, R1.1
- net N$2: now also J2.POS, POWER_SWITCH.1; no longer LED.5, R2.1
- net N$3: now also FUSE.1, J2.NEG; no longer LED.4, R3.1
- net N$5: now also OS2.ANODE, R5.1; no longer GREEN.2, R2.2
- net N$6: now also OS1.ANODE, R3.1; no longer BLUE.2, R1.2
Other:
- moved on the sheet: C1, C2, C3, C4, C5, C6, R2, R3, R4
