File: 2024/PCBs/tsop_PCB_V2.brd (EAGLE design)
At the start: 73.7 x 73.7 mm, 44 parts, among them IC2 CD74HC4067SM96, Q1 BSS138

Commit message: tsop
Parts:
- moved IR16 66.7 mm to (-24.0, 24.0), turned to 135 degrees
- moved IR15 65.7 mm to (-8.80, 32.8), turned to 105 degrees
- moved IR14 64.4 mm to (8.80, 32.8), turned to 75 degrees
- moved IR13 62.8 mm to (24.0, 24.0), turned to 45 degrees
- moved IR12 44.8 mm to (29.4, -17.0), turned to 330 degrees
- moved IR11 41.4 mm to (17.0, -29.4), turned to 300 degrees
- moved IR10 37.8 mm to (0.00, -34.0), turned to 270 degrees
- moved IR9 34.0 mm to (-17.0, -29.4), turned to 240 degrees
- moved IR8 30.1 mm to (-29.4, -17.0), turned to 210 degrees
- moved IR7 26.0 mm to (-34.0, 0.00), turned to 180 degrees
- moved IR6 21.9 mm to (-29.4, 17.0), turned to 150 degrees
- moved IR5 17.6 mm to (-17.0, 29.4), turned to 120 degrees
- moved IR4 13.3 mm to (0.00, 34.0), turned to 90 degrees
- moved IR3 8.88 mm to (17.0, 29.4), turned to 60 degrees
- moved IR2 4.45 mm to (29.4, 17.0), turned to 30 degrees
Connections:
- net I10: no longer IR14.VO, IR16.VO
- net I12: now also IR13.VO
- net I13: now also IR14.VO
- net I14: now also IR15.VO
- net I15: now also IR16.VO
- net I9: no longer IR13.VO, IR15.VO
