File: 2024/PCBs/tsop_PCB_V2.sch (EAGLE design)
At the start: 44 parts, among them IC2 CD74HC4067SM96, Q1 BSS138

Commit message: tsop
Connections:
- net I10: no longer IR14.VO, IR16.VO
- net I12: now also IR13.VO
- net I13: now also IR14.VO
- net I14: now also IR15.VO
- net I15: now also IR16.VO
- net I9: no longer IR13.VO, IR15.VO
Other:
- moved on the sheet: C10, C11, C12, C13, C14, C15, C16, C17, C2, C3, C4, C5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
