File: 2024/PCBs/tsop_PCB_V1.brd (EAGLE design)
At the start: 60 x 60 mm, 84 parts, among them IC2 CD74HC4067SM96, Q1 BSS138

Commit message: tsopV1
Parts:
- removed C11, C13, C3, C5, C7, C9: 100nF, rcl:C0805
- added C30, C31, C32, C33: 1u, rcl:C0805
- added IR13, IR14, IR15, IR16: TSSP58038, TSOP4038:TSOP
- added R41, R44, R47, R50: 10R, rcl:R0805
- added R42, R45, R48, R51: 100k, rcl:R0805
- added R43, R46, R49, R52: 4.7k, rcl:R0805
- C14, C15, C16: value (none) -> 1u
- R10, R13, R7: value (none) -> 4.7k
- R11, R5, R8: value (none) -> 10R
- R12, R6, R9: value (none) -> 100k
- moved R27 10.8 mm to (2.54, 27.3), turned to 90 degrees
- moved R28 7.69 mm to (0.00, 27.3)
- moved IR11 7.00 mm to (16.0, -27.7)
- moved IR12 7.00 mm to (27.7, -16.0)
- moved IR2 7.00 mm to (27.7, 16.0)
- moved IR3 7.00 mm to (16.0, 27.7)
- moved IR5 7.00 mm to (-16.0, 27.7)
- moved IR6 7.00 mm to (-27.7, 16.0)
- moved IR8 7.00 mm to (-27.7, -16.0)
- moved IR9 7.00 mm to (-16.0, -27.7)
- moved IR1 7.00 mm to (32.0, 0.00)
- moved IR10 7.00 mm to (0.00, -32.0)
- moved IR4 7.00 mm to (0.00, 32.0)
- moved IR7 7.00 mm to (-32.0, 0.00)
- moved R26 6.63 mm to (-2.51, 27.3)
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Connections:
- new net N$24: IR13.VS, R41.2
- new net N$28: IR14.VS, R44.2
- new net N$31: IR15.VS, R47.2
- new net N$33: IR16.VS, R50.2
- new net N$35: IR13.VO, R42.2, R43.2
- new net N$37: IR14.VO, R45.2, R46.2
- new net N$38: IR15.VO, R48.2, R49.2
- new net N$39: IR16.VO, R51.2, R52.2
- net +5V: now also R41.1, R43.1, R44.1, R46.1, R47.1, R49.1, R50.1, R52.1; no longer C11.1, C13.1, C3.1, C5.1, C7.1, C9.1
- net GND: now also C30.2, C31.2, C32.2, C33.2, IR13.GND, IR14.GND, IR15.GND, IR16.GND; no longer C11.2, C13.2, C3.2, C5.2, C7.2, C9.2
- net I12: now also C30.1, R42.1
- net I13: now also C31.1, R45.1
- net I14: now also C32.1, R48.1
- net I15: now also C33.1, R51.1
Routing:
- net +5V: track 378.0 -> 0.00 mm, vias 14 -> 0
- net I0: track 55.5 -> 0.00 mm, vias 1 -> 0
- net I1: track 50.7 -> 0.00 mm, vias 1 -> 0
- net I2: track 45.0 -> 0.00 mm, vias 1 -> 0
- net LIGHT_SET_2: track 38.5 -> 0.00 mm
- net I3: track 35.9 -> 0.00 mm, vias 1 -> 0
- net I4: track 34.0 -> 0.00 mm, vias 1 -> 0
- net IR_READ: track 29.5 -> 0.00 mm
- net I5: track 27.6 -> 0.00 mm, vias 1 -> 0
- net LIGHT_SET_3: track 27.4 -> 0.00 mm, vias 1 -> 0
- net I8: track 22.6 -> 0.00 mm, vias 1 -> 0
- net LIGHT_SET_0: track 21.6 -> 0.00 mm, vias 1 -> 0
- net I10: track 21.5 -> 0.00 mm, vias 1 -> 0
- net I11: track 21.2 -> 0.00 mm, vias 1 -> 0
- net I9: track 20.6 -> 0.00 mm, vias 1 -> 0
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Other:
- board size 60 x 60 mm -> 73.7 x 73.7 mm

Commit message: tsopV1
Parts:
- removed BLUE, GREEN, RED: (no value), jumper:SJ
- removed C10, C12, C8: 100nF, rcl:C0805
- removed LED: LTST-G563ZEGBW, LTST-G563ZEGBW:LED_LTST-G563ZEGBW
- removed Q1: BSS138, BSS138:SOT95P240X111-3N
- removed R1, R2, R3: 330R, rcl:R1206
- removed R4: 10K, rcl:R1206
- added C3, C5, C7: 100nF, rcl:C0805
- moved C6 40.3 mm to (-8.89, -20.3), flipped to the top, turned to 60 degrees
- moved C4 21.0 mm to (-13.0, 18.9), flipped to the top, turned to 300 degrees
- moved C15 13.3 mm to (20.9, -18.3), turned to 330 degrees
- moved C17 13.1 mm to (-26.0, -8.43), turned to 210 degrees
- moved R9 11.1 mm to (22.2, -15.9), turned to 330 degrees
- moved R15 10.5 mm to (-24.7, -10.7), turned to 210 degrees
- moved R10 7.59 mm to (23.5, -13.3)
- moved R16 7.10 mm to (-23.5, -13.1)
- moved R14 6.35 mm to (-22.2, -15.4)
- moved R8 5.92 mm to (24.8, -10.8)
- moved C2 5.01 mm to (23.1, 2.54), flipped to the top, turned to 180 degrees
- moved C30 2.02 mm to (13.7, 15.2)
- moved C31 2.01 mm to (4.51, 19.6)
- moved C21 1.80 mm to (-0.64, 15.2)
- moved C25 0.43 mm to (-23.9, 1.65)
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Connections:
- removed net N$1: LED.6, R1.1
- removed net N$2: LED.5, R2.1
- removed net N$3: LED.4, R3.1
- removed net N$4: R3.2, RED.2
- removed net N$5: GREEN.2, R2.2
- removed net N$6: BLUE.2, R1.2
- removed net N$7: BLUE.1, GREEN.1, Q1.2, RED.1
- net +5V: now also C3.1, C5.1, C7.1; no longer C10.1, C12.1, C8.1, Q1.3
- net GND: now also C3.2, C5.2, C7.2; no longer C10.2, C12.2, C8.2, LED.1, LED.2, LED.3, R4.1
- net LED_UP: no longer Q1.1, R4.2
Routing:
- net +5V: track 0.00 -> 262.6 mm, vias 0 -> 17
- net I0: track 0.00 -> 54.7 mm, vias 0 -> 1
- net I1: track 0.00 -> 49.9 mm, vias 0 -> 1
- net I2: track 0.00 -> 45.1 mm, vias 0 -> 1
- net I15: track 0.00 -> 42.8 mm, vias 0 -> 1
- net I14: track 0.00 -> 41.8 mm, vias 0 -> 1
- net I3: track 0.00 -> 40.3 mm, vias 0 -> 1
- net I13: track 0.00 -> 33.2 mm, vias 0 -> 1
- net IR_READ: track 0.00 -> 32.7 mm, vias 0 -> 1
- net I11: track 0.00 -> 32.4 mm, vias 0 -> 1
- net I4: track 0.00 -> 31.3 mm, vias 0 -> 1
- net I12: track 0.00 -> 29.2 mm, vias 0 -> 1
- net I8: track 0.00 -> 27.4 mm, vias 0 -> 1
- net I10: track 0.00 -> 26.7 mm, vias 0 -> 1
- net I9: track 0.00 -> 25.9 mm, vias 0 -> 1
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
Commit message: diera
Other:
- outline, holes or cut-outs redrawn
- board text added: "Fajnor"
- board text added: "LILA"
- board text removed: "STELA"
Changed lines of the file:
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@@
 <drawing>
 <settings>
-<setting alwaysvectorfont="no"/>
+<setting alwaysvectorfont="yes"/>
 <setting verticaltext="up"/>
 </settings>
@@
 </layers>
 <board>
-<fusionsync huburn="a.cGVyc29uYWw6dWUyZmFhODJh" projecturn="a.cGVyc29uYWw6dWUyZmFhODI5IzIwMjIwNTE3NTI2MjM2NDc2" f3durn="urn:adsk.wipprod:dm.lineage:kAxL2zAkQbyg34I5CNIsDA" pcbguid="" lastpulledtime="" lastsyncedchangeguid="" latestrevisionid="3df3374e-0acd-487a-992f-367c32ada1a6" lastsyncedrevisionid="3df3374e-0acd-487a-992f-367c32ada1a6" lastboardhashguid="29aac0d3-9817-73fd-04b3-c0c4eb913779" lastpushedtime="2024-04-02T20:16:43Z" linktopcb3d="true"/>
+<fusionsync huburn="a.cGVyc29uYWw6dWUyZmFhODJh" projecturn="a.cGVyc29uYWw6dWUyZmFhODI5IzIwMjIwNTE3NTI2MjM2NDc2" f3durn="urn:adsk.wipprod:dm.lineage:kAxL2zAkQbyg34I5CNIsDA" pcbguid="" lastpulledtime="" lastsyncedchangeguid="" latestrevisionid="f2628555-97db-43c9-9961-b171493664a6" lastsyncedrevisionid="f2628555-97db-43c9-9961-b171493664a6" lastboardhashguid="e286c036-01b3-ca11-4021-d167c72f9518" lastpushedtime="2024-04-21T20:27:59Z" linktopcb3d="true"/>
 <plain>
 <circle x="0" y="0" radius="36.83" width="0.0254" layer="20"/>
@@
 <hole x="-17.538696875" y="-10.14420625" drill="3"/>
 <text x="2.032" y="-14.0208" size="0.6096" layer="25" font="vector" ratio="20" rot="R180">XLC-CAPTUR</text>
-<text x="2.7432" y="-11.9634" size="1.6764" layer="25" font="vector" ratio="20" rot="R180">STELA</text>
+<text x="1.905" y="-11.938" size="1.6764" layer="25" font="vector" ratio="20" rot="R180">LILA</text>
+<text x="4.318" y="-12.954" size="0.5" layer="25" font="vector" ratio="18" rot="R180">Fajnor</text>
+<wire x1="15.113" y1="-7.874" x2="14.351" y2="-9.144" width="0.1524" layer="20" curve="44.332677"/>
+<wire x1="14.351" y1="-9.144" x2="12.192" y2="-11.049" width="0.1524" layer="20" curve="-79.55787"/>
+<wire x1="12.192" y1="-11.049" x2="7.747" y2="-8.763" width="0.1524" layer="20" curve="-57.721537"/>
+<wire x1="7.747" y1="-8.763" x2="5.588" y2="-6.477" width="0.1524" layer="20" curve="18.880589"/>
+<wire x1="5.588" y1="-6.477" x2="4.699" y2="-2.159" width="0.1524" layer="20" curve="-82.340218"/>
+<wire x1="4.699" y1="-2.159" x2="6.858" y2="0" width="0.1524" layer="20" curve="-30.927091"/>
+<wire x1="6.858" y1="0" x2="10.16" y2="3.81" width="0.1524" layer="20" curve="39.098331"/>
+<wire x1="10.16" y1="3.81" x2="14.097" y2="5.207" width="0.1524" layer="20" curve="-98.19633"/>
+<wire x1="14.097" y1="5.207" x2="14.859" y2="4.699" width="0.1524" layer="20" curve="-8.257149"/>
+<wire x1="14.859" y1="4.699" x2="16.002" y2="3.302" width="0.1524" layer="20" curve="-25.783927"/>
+<wire x1="16.002" y1="3.302" x2="18.669" y2="-0.508" width="0.1524" layer="20" curve="17.189193"/>
+<wire x1="18.669" y1="-0.508" x2="21.844" y2="-3.683" width="0.1524" layer="20" curve="2.82676"/>
+<wire x1="21.844" y1="-3.683" x2="22.86" y2="-8.763" width="0.1524" layer="20" curve="-70.206872"/>
+<wire x1="22.86" y1="-8.763" x2="21.336" y2="-9.017" width="0.1524" layer="20" curve="-113.488318"/>
+<wire x1="21.336" y1="-9.017" x2="20.193" y2="-7.874" width="0.1524" layer="20" curve="4.563604"/>
+<wire x1="20.193" y1="-7.874" x2="16.51" y2="-7.112" width="0.1524" layer="20" curve="62.057646"/>
+<wire x1="15.113" y1="-7.874" x2="16.51" y2="-7.112" width="0.1524" layer="20" curve="-16.518806"/>
 </plain>
 <attributes>
@@
 <wire x1="-2.032" y1="-5.08" x2="-2.267" y2="-4.845" width="0.4064" layer="16"/>
 <via x="-1.143" y="-5.08" extent="1-16" drill="0.35"/>
-<wire x1="3.81" y1="3.81" x2="3.81" y2="3.175" width="0.4064" layer="1"/>
 <wire x1="24.017" y1="2.54" x2="26.355" y2="2.54" width="0.4064" layer="1"/>
 <wire x1="9.4910875" y1="19.476" x2="10.795" y2="21.59" width="0.4064" layer="1"/>
@@
 <wire x1="1.27" y1="-25.72" x2="-12.13461875" y2="-22.9811375" width="1.016" layer="16"/>
 <wire x1="-12.13461875" y1="-22.9811375" x2="-21.98410625" y2="-13.837640625" width="1.016" layer="16"/>
-<wire x1="3.81" y1="6.985" x2="3.81" y2="3.81" width="1.016" layer="1"/>
 <wire x1="3.81" y1="-0.0334125" x2="-0.93579375" y2="-4.77920625" width="1.016" layer="1"/>
 <wire x1="-0.93579375" y1="-4.77920625" x2="-1.18979375" y2="-5.03320625" width="1.016" layer="1"/>
-<wire x1="3.81" y1="3.175" x2="3.81" y2="-0.0334125" width="1.016" layer="1"/>
 <wire x1="-0.93579375" y1="-4.77920625" x2="-2.54" y2="-6.223" width="1.016" layer="1"/>
 <wire x1="-2.54" y1="-6.223" x2="-21.376875" y2="-14.9428" width="1.016" layer="1" curve="-34.294853"/>
@@
 <wire x1="23.942275" y1="-10.32" x2="23.40881875" y2="-11.386909375" width="0.4064" layer="1"/>
 <wire x1="-1.143" y1="-5.08" x2="-0.93579375" y2="-4.77920625" width="0.4064" layer="1"/>
+<wire x1="3.81" y1="6.985" x2="3.81" y2="-0.0334125" width="1.016" layer="1"/>
 </signal>
 <signal name="N$17">
