File: 2024/PCBs/new_horna_podstava.brd (EAGLE design)
At the start: 170 x 163.8 mm, 26 parts, among them J2 XT60-M

Commit message: LOGO
Parts:
- removed BNO085: 4754, 4754:MODULE_4754
- removed C1: 100nF, rcl:C0805
- removed OS1, OS2: (no value), tcrt5000:TCRT5000
- removed R2, R4: 4k7, rcl:R1206
- removed R3, R5: 330R, rcl:R1206
- added C16: (no value), rcl:C0805
- added C18: 1u, rcl:C0805
- added C7, C8: 100nF, rcl:C0805
- added IR1, IR2: TSSP58038, TSOP4038:TSOP
- added JP1: (no value), adafruit:1X06
- added R1: 10K, rcl:R1206
- added R11, R12, R13: (no value), rcl:R0805
- added R17: 10R, rcl:R0805
- added R18: 100k, rcl:R0805
- added R19: 4.7k, rcl:R0805
- added U$1: ROBOCUP_MODULE, ROBOCUP_MODULE:ROBOCUP_MODULE
- added U$10, U$11, U$12, U$3, U$4, U$5, U$6, U$7, U$8, U$9: PAD_MOTORS, PAD_MOTORS:PAD_MOTORS
- added U$2: L298NMOTORDRIVER, l298n motor driver:L298NMOTORDRIVER
- added U1: 2472, 2472:MODULE_2472
- added X1: 332-02, con-garry:332-02
- moved C6 21.7 mm to (2.54, 33.0), turned to 90 degrees
- moved J2 1.55 mm to (0.25, -40.9)
- moved POWER_SWITCH 1.40 mm to (0.00, -52.2)
Connections:
- removed net BALL_CHECK_0: ARDUINO_MEGA.A8, OS1.C, R2.1
- removed net BALL_CHECK_1: ARDUINO_MEGA.A10, OS2.C, R4.1
- removed net N$5: OS2.A, R5.1
- removed net N$6: OS1.A, R3.1
- new net 3VO: U1.2
- new net 5V: ARDUINO_MEGA.5V_1, ARDUINO_MEGA.5V_2, ARDUINO_MEGA.5V_3
- new net BUTTON_KICK: ARDUINO_MEGA.D46, R1.1, X1.2
- new net DIG_OUT: ARDUINO_MEGA.D15, U$1.10
- new net DRIBLER+: U$11.P$2, U$5.P$2
- new net DRIBLER-: U$12.P$2, U$6.P$2
- new net EN1: ARDUINO_MEGA.D8, JP1.1
- new net EN2: ARDUINO_MEGA.D10, JP1.6
- new net I0: ARDUINO_MEGA.A10, C16.1, R12.1
- new net I1: ARDUINO_MEGA.A8, C18.1, R18.1
- new net IN1: ARDUINO_MEGA.D11, JP1.2
- new net IN2: ARDUINO_MEGA.D12, JP1.3
- new net IN3: ARDUINO_MEGA.D13, JP1.4
- new net IN4: ARDUINO_MEGA.D14, JP1.5
- new net KICK+: U$3.P$2, U$9.P$2
- new net KICK-: U$10.P$2, U$4.P$2
- new net N$11: IR2.VS, R17.2
- new net N$23: IR1.VO, R12.2, R13.2
- new net N$27: IR2.VO, R18.2, R19.2
- new net N$9: IR1.VS, R11.2
- net +12V: now also ARDUINO_MEGA.VIN_1, ARDUINO_MEGA.VIN_2, U$7.P$2
- net +5V: now also C7.1, C8.1, R11.1, R13.1, R17.1, R19.1, U1.1, X1.1; no longer ARDUINO_MEGA.5V_1, ARDUINO_MEGA.5V_2, ARDUINO_MEGA.5V_3, BNO085.JP1_1, C1.1, R2.2, R3.2, R4.2, R5.2
- net GND: now also C16.2, C18.2, C7.2, C8.2, IR1.GND, IR2.GND, R1.2, U$1.4, U$8.P$2, U1.3; no longer BNO085.JP1_3, C1.2, OS1.E, OS1.K, OS2.E, OS2.K
- net GYRO_SCL: now also U1.5; no longer BNO085.JP1_4
- net GYRO_SDA: now also U1.4; no longer BNO085.JP1_5
- net N$2: now also U$1.1
Routing:
- net +12V: track 0.00 -> 188.2 mm
- net IN3: track 0.00 -> 123.5 mm, vias 0 -> 3
- net IN1: track 0.00 -> 122.8 mm, vias 0 -> 3
- net +5V: track 482.9 -> 371.1 mm, vias 1 -> 7
- net EN2: track 0.00 -> 111.2 mm, vias 0 -> 4
- net IN4: track 0.00 -> 105.1 mm, vias 0 -> 6
- net IN2: track 0.00 -> 99.0 mm, vias 0 -> 5
- net EN1: track 0.00 -> 94.7 mm, vias 0 -> 4
- net I1: track 0.00 -> 85.0 mm
- net BALL_CHECK_1: track 73.1 -> 0.00 mm
- net BALL_CHECK_0: track 71.8 -> 0.00 mm
- net I0: track 0.00 -> 54.9 mm, vias 0 -> 1
- net DRIBLER+: track 0.00 -> 40.3 mm
- net N$2: track 7.64 -> 45.4 mm
- net KICK-: track 0.00 -> 35.0 mm
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Other:
- board text added: "2024"
- board text removed: "2023"
