File: 2024/PCBs/new_horna_podstava.sch (EAGLE design)
At the start: 26 parts, among them J2 XT60-M

Commit message: LOGO
Parts:
- removed BNO085: 4754, 4754:4754
- removed C1: 100nF, rcl:C-EUC0805
- removed OS1, OS2: (no value), tcrt5000:TCRT5000
- removed R2, R4: 4k7, rcl:R-EU_R1206
- removed R3, R5: 330R, rcl:R-EU_R1206
- added C16: (no value), rcl:C-EUC0805
- added C18: 1u, rcl:C-EUC0805
- added C7, C8: 100nF, rcl:C-EUC0805
- added IR1, IR2: TSSP58038, TSOP4038:TSOP4038
- added JP1: (no value), adafruit:PINHD-1X6
- added R1: 10K, rcl:R-EU_R1206
- added R11, R12, R13: (no value), rcl:R-EU_R0805
- added R17: 10R, rcl:R-EU_R0805
- added R18: 100k, rcl:R-EU_R0805
- added R19: 4.7k, rcl:R-EU_R0805
- added U$1: ROBOCUP_MODULE, ROBOCUP_MODULE:ROBOCUP_MODULE
- added U$10, U$11, U$12, U$3, U$4, U$5, U$6, U$7, U$8, U$9: PAD_MOTORS, PAD_MOTORS:PAD_MOTORS
- added U$2: L298NMOTORDRIVER, l298n motor driver:L298NMOTORDRIVER
- added U1: 2472, 2472:2472
- added X1: 332-02, con-garry:332-02
Connections:
- removed net BALL_CHECK_0: ARDUINO_MEGA.A8, OS1.COLLECTOR, R2.1
- removed net BALL_CHECK_1: ARDUINO_MEGA.A10, OS2.COLLECTOR, R4.1
- removed net N$5: OS2.ANODE, R5.1
- removed net N$6: OS1.ANODE, R3.1
- new net BUTTON_KICK: ARDUINO_MEGA.D46, R1.1, X1-2.S
- new net DIG_OUT: ARDUINO_MEGA.D15, U$1.6
- new net DRIBLER+: U$11.P$1, U$5.P$1
- new net DRIBLER-: U$12.P$1, U$6.P$1
- new net EN1: ARDUINO_MEGA.D8, JP1.1
- new net EN2: ARDUINO_MEGA.D10, JP1.6
- new net I0: ARDUINO_MEGA.A10, C16.1, R12.1
- new net I1: ARDUINO_MEGA.A8, C18.1, R18.1
- new net IN1: ARDUINO_MEGA.D11, JP1.2
- new net IN2: ARDUINO_MEGA.D12, JP1.3
- new net IN3: ARDUINO_MEGA.D13, JP1.4
- new net IN4: ARDUINO_MEGA.D14, JP1.5
- new net KICK+: U$3.P$1, U$9.P$1
- new net KICK-: U$10.P$1, U$4.P$1
- new net N$11: IR2.VS, R17.2
- new net N$23: IR1.VO, R12.2, R13.2
- new net N$27: IR2.VO, R18.2, R19.2
- new net N$9: IR1.VS, R11.2
- net +12V: now also ARDUINO_MEGA.VIN, U$7.P$1
- net +5V: now also C7.1, C8.1, R11.1, R13.1, R17.1, R19.1, U1.VIN, X1-1.S; no longer ARDUINO_MEGA.5V, BNO085.VIN, C1.1, R2.2, R3.2, R4.2, R5.2
- net GND: now also C16.2, C18.2, C7.2, C8.2, IR1.GND, IR2.GND, R1.2, U$1.10, U$8.P$1, U1.GND; no longer BNO085.GND, C1.2, OS1.CATHODE, OS1.EMITTER, OS2.CATHODE, OS2.EMITTER
- net GYRO_SCL: now also U1.SCL; no longer BNO085.SCL
- net GYRO_SDA: now also U1.SDA; no longer BNO085.SDA
- net N$2: now also U$1.7
